Commit message: add cylinder base do model.

File: ROS/open_base/xacro/main.urdf.xacro (robot description, xacro)
@@ -5,5 +5,12 @@
 >
 	<xacro:include filename="$(find open_base)/xacro/rim.urdf.xacro"/>
-	<link name="origin_link"/>
+	<!-- Used for fixing robot to Gazebo 'base_link' -->
+  <link name="world"/>
+  <joint name="fixed" type="fixed">
+    <parent link="world"/>
+    <child link="base_link"/>
+		<origin xyz="0 0 0.07" rpy="3.14 0 0 "	/>
+  </joint>
+	<!-- <link name="origin_link"/> -->
 	<link name="base_link">
 	<inertial>
@@ -32,5 +39,5 @@
 	</collision>
 	</link>
-	<joint
+	<!-- <joint
 		name="base_joint"
 		type="fixed"
@@ -38,8 +45,38 @@
 		<parent link="origin_link" />
 		<child link="base_link" />
-		<origin
-			xyz="0 0 0.01905"
-		/>
+		<origin xyz="0 0 0.01905" rpy="3.14 0 0 "	/>
+	</joint> -->
+	<joint 	name="body_joint"	type="fixed" >
+		<parent link="base_link"/>
+		<child link="body_link"/>
+		<axis xyz="0 0 1"/>
+		<origin xyz="0 0 0.01905"/>
 	</joint>
+	<link name="body_link">
+		<inertial>
+			<mass value="0.5"/>
+			<inertia
+				ixx="1"
+				ixy="0"
+				ixz="0"
+				iyy="1"
+				iyz="0"
+				izz="1"
+			/>
+		</inertial>
+		<visual>
+			<geometry>
+				<cylinder radius="0.02" length="0.05"/>
+			</geometry>
+			<material name="base_material">
+				<color rgba="1 1 1 1"/>
+			</material>
+		</visual>
+		<collision>
+			<geometry>
+				<cylinder radius="0.02" length="0.05"/>
+			</geometry>
+		</collision>
+	</link>
 	<xacro:rim_macro
 		name="left"
